File: hardware/epaper-breakout/epaper-breakout.kicad_pcb (KiCad board)
At the start: 2 copper layers, 100 x 40.5 mm, 90 parts, among them J1 XF2M-3315-1A, J2 C10418, J3 Conn_02x06_Counter_Clockwise, J4 ED060SC4, J5 Conn_01x01_Male, J6 Conn_01x01_Male, Q1 AO3401A, Q2 AO3401A, Q3 MMBT3904, Q4 MMBT3904, Q5 AO3401A, Q6 MMBT3904, U1 MCP1700-3302E_SOT23, U10 ED060SC7, U11 TP4056, U12 CH340C, U2 LT1945, U3 LT1945, U4 XC6206PxxxMR, U5 ESP32-WROVER, U6 ED060XC5, U7 LM358, U8 74HC4094-normal, U9 MCP9700AT-ETT

Commit message: saved in new format
Parts:
- removed H1, H2, H3: MountingHole, MountingHole:MountingHole_2.2mm_M2
- removed J3: Conn_02x06_Counter_Clockwise, Connector_PinHeader_2.54mm:PinHeader_2x06_P2.54mm_Vertical
- removed J4: ED060SC4, epaper-breakout:HRS_FH26W-39S-0.3SHW(60)
- removed JP_TEMP1: Jumper, Jumper:SolderJumper-2_P1.3mm_Bridged2Bar_RoundedPad1.0x1.5mm
- removed U10: ED060SC7, epaper-breakout:AXT334124
- removed U6: ED060XC5, epaper-breakout:X05A20H34G
- removed U7: LM358, Package_SO:SOP-8_3.76x4.96mm_P1.27mm
- removed U9: MCP9700AT-ETT, Package_TO_SOT_SMD:SOT-23
- moved J1 2.82 mm to (115.0, 35.1)
- moved U3 1.34 mm to (62.2, 44.6)
- moved U2 1.23 mm to (47.2, 29.0)
- moved U12 1.16 mm to (29.2, 37.2)
- moved U8 1.13 mm to (76.1, 25.0)
- moved U11 0.70 mm to (42.7, 47.8)
- moved U5 0.45 mm to (96.3, 26.4)
Connections:
- J1 pad 2: (no net) -> unconnected-(J1-Pad2)
- J1 pad 21: (no net) -> unconnected-(J1-Pad21)
- J1 pad 23: (no net) -> unconnected-(J1-Pad23)
- J1 pad 25: (no net) -> unconnected-(J1-Pad25)
- J1 pad 27: (no net) -> unconnected-(J1-Pad27)
- J1 pad 34: (no net) -> unconnected-(J1-Pad34)
- J1 pad 35: (no net) -> unconnected-(J1-Pad35)
- J1 pad 4: (no net) -> unconnected-(J1-Pad4)
- J1 pad 6: (no net) -> unconnected-(J1-Pad6)
- J2 pad 4: (no net) -> unconnected-(J2-Pad4)
- U11 pad 9: (no net) -> unconnected-(U11-Pad9)
- U12 pad 10: (no net) -> unconnected-(U12-Pad10)
- U12 pad 11: (no net) -> unconnected-(U12-Pad11)
- U12 pad 12: (no net) -> unconnected-(U12-Pad12)
- U12 pad 15: (no net) -> unconnected-(U12-Pad15)
- U12 pad 7: (no net) -> unconnected-(U12-Pad7)
- U12 pad 8: (no net) -> unconnected-(U12-Pad8)
- U12 pad 9: (no net) -> unconnected-(U12-Pad9)
- U5 pad 17: (no net) -> unconnected-(U5-Pad17)
- U5 pad 18: (no net) -> unconnected-(U5-Pad18)
- U5 pad 19: (no net) -> unconnected-(U5-Pad19)
- U5 pad 20: (no net) -> unconnected-(U5-Pad20)
- U5 pad 21: (no net) -> unconnected-(U5-Pad21)
- U5 pad 22: (no net) -> unconnected-(U5-Pad22)
- U5 pad 27: (no net) -> unconnected-(U5-Pad27)
- U5 pad 28: (no net) -> unconnected-(U5-Pad28)
- U5 pad 32: (no net) -> unconnected-(U5-Pad32)
- U8 pad 10: (no net) -> unconnected-(U8-Pad10)
- U8 pad 9: (no net) -> unconnected-(U8-Pad9)
Routing:
- net GND: track 262.0 -> 0.00 mm, vias 132 -> 0
- net /-20V: track 188.8 -> 0.00 mm, vias 8 -> 0
- net EPD_VDD: track 184.5 -> 0.00 mm, vias 12 -> 0
- net /+22V: track 178.2 -> 0.00 mm, vias 6 -> 0
- net /EP_VCOM: track 177.6 -> 0.00 mm, vias 8 -> 0
- net /EP_STV: track 152.7 -> 0.00 mm, vias 5 -> 0
- net /EP_CKV: track 149.6 -> 0.00 mm, vias 6 -> 0
- net /-15V: track 147.9 -> 0.00 mm, vias 9 -> 0
- net /EP_MODE: track 140.8 -> 0.00 mm, vias 4 -> 0
- net /15V: track 139.3 -> 0.00 mm, vias 8 -> 0
- net /+3.3V: track 135.8 -> 0.00 mm, vias 4 -> 0
- net /EP_OE: track 133.2 -> 0.00 mm, vias 8 -> 0
- net /EP_D6: track 123.6 -> 0.00 mm, vias 6 -> 0
- net /EP_D7: track 121.4 -> 0.00 mm, vias 4 -> 0
- net /EP_D5: track 113.3 -> 0.00 mm, vias 4 -> 0
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- removed copper zone on B.Cu, net GND
- removed copper zone on F.Cu, net GND
Other:
- net class Default removed
- board text removed: "ED060SC4"
- board text removed: "ED060SC7"
- board text removed: "ED060XC5"
